File: solar_emulator.kicad_sch (KiCad schematic)
At the start: 69 parts, among them J1 USB_C_Receptacle_USB2.0_16P, J2 Conn_01x02, J3 Conn_01x02, J4 Conn_01x02, J5 Conn_01x02, J6 Conn_01x03, J7 Conn_01x04, Q1 IRFZ44N, Q2 IRFZ44N, Q3 IRFZ44N, Q4 IRFZ44N, Q5 IRFZ44N, Q6 IRFZ44N, Q7 IRFZ44N, Q8 IRFZ44N, SW1 SW_Push, SW2 SW_Push, U1 ESP32-S3-WROOM-1, U2 LD1117S33TR_SOT223, U3 HIP4081AIPZ, U4 HIP4081AIPZ, U5 LM393, U6 LM393

Commit message: implement +12V copper fills, routing basically complete
Connections:
- net AHI1: now also U1.23 (GPIO21); no longer U1.4 (GPIO4/TOUCH4/ADC1_CH3)
- net AHI2: now also U1.15 (GPIO3/TOUCH3/ADC1_CH2); no longer U1.12 (GPIO8/TOUCH8/ADC1_CH7/SUBSPICS1)
- net ALI1: now also U1.24 (GPIO47/SPICLK_P/SUBSPICLK_P_DIFF); no longer U1.15 (GPIO3/TOUCH3/ADC1_CH2)
- net ALI2: now also U1.16 (GPIO46); no longer U1.7 (GPIO7/TOUCH7/ADC1_CH6)
- net BHI1: now also U1.26 (GPIO45); no longer U1.39 (GPIO1/TOUCH1/ADC1_CH0)
- net BHI2: now also U1.18 (GPIO10/TOUCH10/ADC1_CH9/FSPICS0/FSPIIO4/SUBSPICS0); no longer U1.5 (GPIO5/TOUCH5/ADC1_CH4)
- net BLI1: now also U1.25 (GPIO48/SPICLK_N/SUBSPICLK_N_DIFF); no longer U1.38 (GPIO2/TOUCH2/ADC1_CH1)
- net BLI2: now also U1.17 (GPIO9/TOUCH9/ADC1_CH8/FSPIHD/SUBSPIHD); no longer U1.6 (GPIO6/TOUCH6/ADC1_CH5)
- net LIMIT1: now also U1.38 (GPIO2/TOUCH2/ADC1_CH1); no longer U1.18 (GPIO10/TOUCH10/ADC1_CH9/FSPICS0/FSPIIO4/SUBSPICS0)
- net LIMIT2: now also U1.39 (GPIO1/TOUCH1/ADC1_CH0); no longer U1.19 (GPIO11/TOUCH11/ADC2_CH0/FSPID/FSPIIO5/SUBSPID)
- net SERVO: now also U1.30 (SPIDQS/GPIO37/FSPIQ/SUBSPIQ); no longer U1.17 (GPIO9/TOUCH9/ADC1_CH8/FSPIHD/SUBSPIHD)
Changed lines of the file:
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@@
 	)
 	(no_connect
-		(at 114.3 82.55)
+		(at 114.3 49.53)
 	)
 	(no_connect
@@
 	)
 	(no_connect
-		(at 114.3 87.63)
+		(at 114.3 52.07)
 	)
 	(no_connect
-		(at 114.3 95.25)
+		(at 114.3 67.31)
 	)
 	(no_connect
-		(at 114.3 92.71)
+		(at 114.3 59.69)
 	)
 	(no_connect
@@
 	)
 	(no_connect
-		(at 114.3 90.17)
+		(at 114.3 57.15)
 	)
 	(no_connect
@@
 	)
 	(no_connect
+		(at 114.3 54.61)
+	)
+	(no_connect
 		(at 114.3 72.39)
 	)
@@
 	)
 	(no_connect
-		(at 22.86 95.25)
-	)
-	(no_connect
 		(at 114.3 77.47)
 	)
@@
 	(global_label "LIMIT1"
 		(shape input)
-		(at 114.3 64.77 0)
+		(at 114.3 44.45 0)
 		(fields_autoplaced yes)
 		(effects
@@
 		)
 		(property "Intersheetrefs" "${INTERSHEET_REFS}"
-			(at 123.1514 64.77 0)
+			(at 121.3976 44.45 0)
 			(hide yes)
 			(show_name no)
@@
 	(global_label "BHI2"
 		(shape input)
-		(at 114.3 52.07 0)
+		(at 114.3 64.77 0)
 		(fields_autoplaced yes)
 		(effects
@@
 		)
 		(property "Intersheetrefs" "${INTERSHEET_REFS}"
-			(at 121.7 52.07 0)
+			(at 121.7 64.77 0)
 			(hide yes)
 			(show_name no)
@@
 	(global_label "ALI2"
 		(shape input)
-		(at 114.3 57.15 0)
+		(at 114.3 90.17 0)
 		(fields_autoplaced yes)
 		(effects
@@
 		)
 		(property "Intersheetrefs" "${INTERSHEET_REFS}"
-			(at 121.2162 57.15 0)
+			(at 121.2162 90.17 0)
 			(hide yes)
 			(show_name no)
@@
 	(global_label "BLI2"
 		(shape input)
-		(at 114.3 54.61 0)
+		(at 114.3 62.23 0)
 		(fields_autoplaced yes)
 		(effects
@@
 		)
 		(property "Intersheetrefs" "${INTERSHEET_REFS}"
-			(at 121.3976 54.61 0)
+			(at 121.3976 62.23 0)
 			(hide yes)
 			(show_name no)
@@
 	(global_label "BLI1"
 		(shape input)
-		(at 114.3 44.45 0)
+		(at 114.3 95.25 0)
 		(fields_autoplaced yes)
 		(effects
@@
 		)
 		(property "Intersheetrefs" "${INTERSHEET_REFS}"
-			(at 121.3976 44.45 0)
+			(at 123.1514 95.25 0)
 			(hide yes)
 			(show_name no)
@@
 	(global_label "AHI2"
 		(shape input)
-		(at 114.3 59.69 0)
+		(at 114.3 46.99 0)
 		(fields_autoplaced yes)
 		(effects
@@
 		)
 		(property "Intersheetrefs" "${INTERSHEET_REFS}"
-			(at 121.5186 59.69 0)
+			(at 121.5186 46.99 0)
 			(hide yes)
 			(show_name no)
@@
 	(global_label "AHI1"
 		(shape input)
-		(at 114.3 49.53 0)
+		(at 114.3 82.55 0)
 		(fields_autoplaced yes)
 		(effects
@@
 		)
 		(property "Intersheetrefs" "${INTERSHEET_REFS}"
-			(at 121.5186 49.53 0)
+			(at 121.5186 82.55 0)
 			(hide yes)
 			(show_name no)
@@
 	(global_label "ALI1"
 		(shape input)
-		(at 114.3 46.99 0)
+		(at 114.3 92.71 0)
 		(fields_autoplaced yes)
 		(effects
@@
 		)
 		(property "Intersheetrefs" "${INTERSHEET_REFS}"
-			(at 121.2162 46.99 0)
+			(at 121.2162 92.71 0)
 			(hide yes)
 			(show_name no)
@@
 	(global_label "BHI1"
 		(shape input)
-		(at 114.3 41.91 0)
+		(at 114.3 87.63 0)
 		(fields_autoplaced yes)
 		(effects
@@
 		)
 		(property "Intersheetrefs" "${INTERSHEET_REFS}"
-			(at 121.7 41.91 0)
+			(at 123.1514 87.63 0)
 			(hide yes)
 			(show_name no)
@@
 	(global_label "SERVO"
 		(shape input)
-		(at 114.3 62.23 0)
+		(at 22.86 95.25 180)
 		(fields_autoplaced yes)
 		(effects
@@
 				(size 1.27 1.27)
 			)
-			(justify left)
+			(justify right)
 		)
 		(property "Intersheetrefs" "${INTERSHEET_REFS}"
-			(at 123.3328 62.23 0)
+			(at 13.8272 95.25 0)
 			(hide yes)
 			(show_name no)
@@
 					(size 1.27 1.27)
 				)
-				(justify left)
+				(justify right)
 			)
 		)
@@
 	(global_label "LIMIT2"
 		(shape input)
-		(at 114.3 67.31 0)
+		(at 114.3 41.91 0)
 		(fields_autoplaced yes)
 		(effects
@@
 		)
 		(property "Intersheetrefs" "${INTERSHEET_REFS}"
-			(at 123.1514 67.31 0)
+			(at 121.7 41.91 0)
 			(hide yes)
 			(show_name no)

Commit message: separate 5V servo and +5V usb
Connections:
- net +5V: no longer J4.2 (Pin_2), J6.2 (Pin_2)
- new net 5V: J4.2 (Pin_2), J6.2 (Pin_2)
Changed lines of the file:
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@@
 	)
 	(symbol
+		(lib_id "SparkFun-PowerSymbol:5V")
+		(at 124.46 165.1 0)
+		(unit 1)
+		(body_style 1)
+		(exclude_from_sim no)
+		(in_bom yes)
+		(on_board yes)
+		(in_pos_files yes)
+		(dnp no)
+		(fields_autoplaced yes)
+		(property "Reference" "#PWR01"
+			(at 124.46 168.91 0)
+			(hide yes)
+			(show_name no)
+			(do_not_autoplace no)
+			(effects
+				(font
+					(size 1.27 1.27)
+				)
+			)
+		)
+		(property "Value" "5V"
+			(at 124.46 161.29 0)
+			(show_name no)
+			(do_not_autoplace yes)
+			(effects
+				(font
+					(size 1.27 1.27)
+				)
+			)
+		)
+		(property "Footprint" ""
+			(at 124.46 165.1 0)
+			(hide yes)
+			(show_name no)
+			(do_not_autoplace no)
+			(effects
+				(font
+					(size 1.27 1.27)
+				)
+			)
+		)
+		(property "Datasheet" ""
+			(at 124.46 165.1 0)
+			(hide yes)
+			(show_name no)
+			(do_not_autoplace no)
+			(effects
+				(font
+					(size 1.27 1.27)
+				)
+			)
+		)
+		(property "Description" "Power symbol creates a global label with name \"5V\""
+			(at 124.46 171.45 0)
+			(hide yes)
+			(show_name no)
+			(do_not_autoplace no)
+			(effects
+				(font
+					(size 1.27 1.27)
+				)
+			)
+		)
+		(pin "1"
+		)
+		(instances
+			(project "solar_emulator"
+				(path "/d8ff8312-ce26-4905-abd5-48c35bcc1ef8"
+					(reference "#PWR01")
+					(unit 1)
+				)
+			)
+		)
+	)
+	(symbol
 		(lib_id "power:GND")
 		(at 123.19 171.45 0)
@@
 	)
 	(symbol
+		(lib_id "SparkFun-PowerSymbol:5V")
+		(at 168.91 154.94 0)
+		(unit 1)
+		(body_style 1)
+		(exclude_from_sim no)
+		(in_bom yes)
+		(on_board yes)
+		(in_pos_files yes)
+		(dnp no)
+		(fields_autoplaced yes)
+		(property "Reference" "#PWR04"
+			(at 168.91 158.75 0)
+			(hide yes)
+			(show_name no)
+			(do_not_autoplace no)
+			(effects
+				(font
+					(size 1.27 1.27)
+				)
+			)
+		)
+		(property "Value" "5V"
+			(at 168.91 151.13 0)
+			(show_name no)
+			(do_not_autoplace yes)
+			(effects
+				(font
+					(size 1.27 1.27)
+				)
+			)
+		)
+		(property "Footprint" ""
+			(at 168.91 154.94 0)
+			(hide yes)
+			(show_name no)
+			(do_not_autoplace no)
+			(effects
+				(font
+					(size 1.27 1.27)
+				)
+			)
+		)
+		(property "Datasheet" ""
+			(at 168.91 154.94 0)
+			(hide yes)
+			(show_name no)
+			(do_not_autoplace no)
+			(effects
+				(font
+					(size 1.27 1.27)
+				)
+			)
+		)
+		(property "Description" "Power symbol creates a global label with name \"5V\""
+			(at 168.91 161.29 0)
+			(hide yes)
+			(show_name no)
+			(do_not_autoplace no)
+			(effects
+				(font
+					(size 1.27 1.27)
+				)
+			)
+		)
+		(pin "1"
+		)
+		(instances
+			(project "solar_emulator"
+				(path "/d8ff8312-ce26-4905-abd5-48c35bcc1ef8"
+					(reference "#PWR04")
+					(unit 1)
+				)
+			)
+		)
+	)
+	(symbol
 		(lib_id "Device:R")
 		(at 154.94 69.85 0)
@@
 	)
 	(symbol
-		(lib_id "power:+5V")
-		(at 168.91 154.94 0)
-		(unit 1)
-		(body_style 1)
-		(exclude_from_sim no)
-		(in_bom yes)
-		(on_board yes)
-		(in_pos_files yes)
-		(dnp no)
-		(fields_autoplaced yes)
-		(property "Reference" "#PWR025"
-			(at 168.91 158.75 0)
-			(hide yes)
-			(show_name no)
-			(do_not_autoplace no)
-			(effects
-				(font
-					(size 1.27 1.27)
-				)
-			)
-		)
-		(property "Value" "+5V"
-			(at 168.91 149.86 0)
-			(show_name no)
-			(do_not_autoplace no)
-			(effects
-				(font
-					(size 1.27 1.27)
-				)
-			)
-		)
-		(property "Footprint" ""
-			(at 168.91 154.94 0)
-			(hide yes)
-			(show_name no)
-			(do_not_autoplace no)
-			(effects
-				(font
-					(size 1.27 1.27)
-				)
-			)
-		)
-		(property "Datasheet" ""
-			(at 168.91 154.94 0)
-			(hide yes)
-			(show_name no)
-			(do_not_autoplace no)
-			(effects
-				(font
-					(size 1.27 1.27)
-				)
-			)
-		)
-		(property "Description" "Power symbol creates a global label with name \"+5V\""
-			(at 168.91 154.94 0)
-			(hide yes)
-			(show_name no)
-			(do_not_autoplace no)
-			(effects
-				(font
-					(size 1.27 1.27)
-				)
-			)
-		)
-		(pin "1"
-		)
-		(instances
-			(project "solar_emulator"
-				(path "/d8ff8312-ce26-4905-abd5-48c35bcc1ef8"
-					(reference "#PWR025")
-					(unit 1)
-				)
-			)
-		)
-	)
-	(symbol
 		(lib_id "power:+3V3")
 		(at 68.58 19.05 0)
@@
 					(unit 1)
 				)
-			)
-		)
-	)
-	(symbol
-		(lib_id "power:+5V")
-		(at 124.46 165.1 0)
-		(unit 1)
-		(body_style 1)
-		(exclude_from_sim no)
-		(in_bom yes)
-		(on_board yes)
-		(in_pos_files yes)
-		(dnp no)
-		(fields_autoplaced yes)
-		(property "Reference" "#PWR019"
-			(at 124.46 168.91 0)
-			(hide yes)
-			(show_name no)
-			(do_not_autoplace no)
-			(effects
-				(font
-					(size 1.27 1.27)
-				)
-			)
-		)
-		(property "Value" "+5V"
-			(at 124.46 160.02 0)
-			(show_name no)
-			(do_not_autoplace no)
-			(effects
-				(font
-					(size 1.27 1.27)
-				)
-			)
-		)
-		(property "Footprint" ""
-			(at 124.46 165.1 0)
-			(hide yes)
-			(show_name no)
-			(do_not_autoplace no)
-			(effects
-				(font
-					(size 1.27 1.27)
-				)
-			)
-		)
-		(property "Datasheet" ""
-			(at 124.46 165.1 0)
-			(hide yes)
-			(show_name no)
-			(do_not_autoplace no)
-			(effects
-				(font
-					(size 1.27 1.27)
-				)
-			)
-		)
-		(property "Description" "Power symbol creates a global label with name \"+5V\""
-			(at 124.46 165.1 0)
-			(hide yes)
-			(show_name no)
-			(do_not_autoplace no)
-			(effects
-				(font
-					(size 1.27 1.27)
-				)
-			)
-		)
-		(pin "1"
-		)
-		(instances
-			(project "solar_emulator"
-				(path "/d8ff8312-ce26-4905-abd5-48c35bcc1ef8"
-					(reference "#PWR019")
-					(unit 1)
-				)

Commit message: Organize schematic in to respective groupings
most footprints change from THT to SMT

this commit still contains THT components on pcb

plan to re design board
Parts:
- added C12: 10u, Capacitor_SMD:C_0603_1608Metric_Pad1.08x0.95mm_HandSolder, symbol Device:C
- added F1: Fuse_Small, symbol Device:Fuse_Small
- added U7: USBLC6-2SC6, Package_TO_SOT_SMD:SOT-23-6, symbol Power_Protection:USBLC6-2SC6
- C1, C4: footprint Capacitor_THT:C_Disc_D9.0mm_W2.5mm_P5.00mm -> Capacitor_SMD:C_0603_1608Metric_Pad1.08x0.95mm_HandSolder
- C10, C11, C5, C6, C7, C8, C9: footprint Capacitor_THT:C_Disc_D4.7mm_W2.5mm_P5.00mm -> Capacitor_SMD:C_0603_1608Metric_Pad1.08x0.95mm_HandSolder
- C2, C3: footprint Capacitor_THT:C_Disc_D6.0mm_W2.5mm_P5.00mm -> Capacitor_SMD:C_0603_1608Metric_Pad1.08x0.95mm_HandSolder
- J2, J3, J4, J5: footprint Connector_PinHeader_2.54mm:PinHeader_1x02_P2.54mm_Vertical -> Connector_JST:JST_PH_B2B-PH-K_1x02_P2.00mm_Vertical
- J6: footprint Connector_PinHeader_2.54mm:PinHeader_1x03_P2.54mm_Vertical -> Connector_JST:JST_PH_B3B-PH-K_1x03_P2.00mm_Vertical
- J7: footprint Connector_PinHeader_2.54mm:PinHeader_1x04_P2.54mm_Vertical -> Connector_JST:JST_PH_B4B-PH-K_1x04_P2.00mm_Vertical
- R10, R11, R12, R13, R14, R15, R16, R17, R18, R19, R20, R21, R22, R23, R24, R27, R28, R29, R30, R4, R5, R6, R7, R8, R9: footprint Resistor_THT:R_Axial_DIN0207_L6.3mm_D2.5mm_P10.16mm_Horizontal -> Resistor_SMD:R_0805_2012Metric_Pad1.20x1.40mm_HandSolder
- R25, R26: footprint Resistor_THT:R_Axial_DIN0207_L6.3mm_D2.5mm_P15.24mm_Horizontal -> Resistor_SMD:R_0805_2012Metric_Pad1.20x1.40mm_HandSolder
Connections:
- net +5V: now also F1.2; no longer J1.A4 (VBUS), J1.A9 (VBUS), J1.B4 (VBUS), J1.B9 (VBUS)
- net D+: now also U7.3 (I/O2); no longer U1.14 (GPIO20/U1CTS/ADC2_CH9/CLK_OUT1/USB_D+)
- net D-: now also U7.1 (I/O1); no longer U1.13 (GPIO19/U1RTS/ADC2_CH8/CLK_OUT2/USB_D-)
- net GND: now also C12.2, U7.2 (GND)
- new net USB_D+: U7.4 (I/O2)
- new net USB_D-: U7.6 (I/O1)
- new net USB_DM: U1.13 (GPIO19/U1RTS/ADC2_CH8/CLK_OUT2/USB_D-)
- new net USB_DP: U1.14 (GPIO20/U1CTS/ADC2_CH9/CLK_OUT1/USB_D+)
- new net VBUS: C12.1, F1.1, J1.A4 (VBUS), J1.A9 (VBUS), J1.B4 (VBUS), J1.B9 (VBUS), U7.5 (VBUS)
Other:
- note added: "COMP 1"
- note added: "COMP 2"
- note added: "Connectors"
- note added: "ESD Protection"
- note added: "ESP32"
- note added: "Motor Driver 1"
- note added: "Motor Driver 2"
- note added: "Mounting Holes"
- note added: "USB-C"
- moved on the sheet: C5, H1, H2, H3, H4, J2, J3, J4, J5, J6, J7, R6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

Commit message: PCB component layout complete, possible refinement needed
Parts:
- D4, D5, D6, D7: footprint Diode_THT:D_DO-41_SOD81_P10.16mm_Horizontal -> Diode_SMD:D_SOD-123
- F1: footprint (none) -> Fuse:Fuse_1206_3216Metric_Pad1.42x1.75mm_HandSolder
Connections:
- net USB_DM is gone; now on net USB_D-: U1.13 (GPIO19/U1RTS/ADC2_CH8/CLK_OUT2/USB_D-)
- net USB_DP is gone; now on net USB_D+: U1.14 (GPIO20/U1CTS/ADC2_CH9/CLK_OUT1/USB_D+)
Other:
- note added: "Regulator"
