File: _restore_backup_2026-08-15T16-14-33-728/solar_emulator.kicad_sch (KiCad schematic)
At the start: 80 parts, among them J1 USB_C_Receptacle_USB2.0_16P, J2 Conn_01x02, J3 Conn_01x02, J4 Conn_01x02, J5 Conn_01x02, J6 Conn_01x03, J7 Conn_01x04, Q1 IRFZ44N, Q2 IRFZ44N, Q3 IRFZ44N, Q4 IRFZ44N, Q5 IRFZ44N, Q6 IRFZ44N, Q7 IRFZ44N, Q8 IRFZ44N, SW1 SW_Push, SW2 SW_Push, U1 ESP32-S3-WROOM-1, U2 LD1117S33TR_SOT223, U3 HIP4081AIPZ, U4 HIP4081AIPZ, U5 LM393, U6 LM393, U7 USBLC6-2SC6

Commit message: add edge cuts to the pcb
Parts:
- removed C12: 10u, Capacitor_SMD:C_0603_1608Metric_Pad1.08x0.95mm_HandSolder, symbol Device:C
- removed D1, D10, D11, D12, D2, D3, D8, D9: D_Zener, Diode_SMD:D_SOD-123, symbol Device:D_Zener
- removed F1: Fuse_Small, Fuse:Fuse_1206_3216Metric_Pad1.42x1.75mm_HandSolder, symbol Device:Fuse_Small
- removed U7: USBLC6-2SC6, Package_TO_SOT_SMD:SOT-23-6, symbol Power_Protection:USBLC6-2SC6
- C1, C4: footprint Capacitor_SMD:C_0603_1608Metric_Pad1.08x0.95mm_HandSolder -> Capacitor_THT:C_Disc_D9.0mm_W2.5mm_P5.00mm
- C10, C11, C5, C6, C7, C8, C9: footprint Capacitor_SMD:C_0603_1608Metric_Pad1.08x0.95mm_HandSolder -> Capacitor_THT:C_Disc_D4.7mm_W2.5mm_P5.00mm
- C2, C3: footprint Capacitor_SMD:C_0603_1608Metric_Pad1.08x0.95mm_HandSolder -> Capacitor_THT:C_Disc_D6.0mm_W2.5mm_P5.00mm
- D4, D5, D6, D7: footprint Diode_SMD:D_SOD-123 -> Diode_THT:D_DO-41_SOD81_P10.16mm_Horizontal
- R10, R11, R12, R13, R14, R15, R16, R17, R18, R19, R20, R21, R22, R23, R24, R27, R28, R29, R30, R4, R5, R6, R7, R8, R9: footprint Resistor_SMD:R_0805_2012Metric_Pad1.20x1.40mm_HandSolder -> Resistor_THT:R_Axial_DIN0207_L6.3mm_D2.5mm_P10.16mm_Horizontal
- R25, R26: footprint Resistor_SMD:R_0805_2012Metric_Pad1.20x1.40mm_HandSolder -> Resistor_THT:R_Axial_DIN0207_L6.3mm_D2.5mm_P15.24mm_Horizontal
Connections:
- net USB_D+ is gone; now on net D+: U1.14 (GPIO20/U1CTS/ADC2_CH9/CLK_OUT1/USB_D+)
- net USB_D- is gone; now on net D-: U1.13 (GPIO19/U1RTS/ADC2_CH8/CLK_OUT2/USB_D-)
- net VBUS is gone; now on net +5V: J1.A4 (VBUS), J1.A9 (VBUS), J1.B4 (VBUS), J1.B9 (VBUS)
Other:
- note removed: "COMP 1"
- note removed: "COMP 2"
- note removed: "Connectors"
- note removed: "ESD Protection"
- note removed: "ESP32"
- note removed: "Motor Driver 1"
- note removed: "Motor Driver 2"
- note removed: "Mounting Holes"
- note removed: "Regulator"
- note removed: "USB-C"
- moved on the sheet: C5, H1, H2, H3, H4, J2, J3, J4, J5, J6, J7, R6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
